File: FLC100_pcb/FLC100_pcb.kicad_pcb (KiCad board)
At the start: 2 copper layers, 99 x 69 mm, 70 parts, among them SW2 DSIC01LS-P_C600988, SW3 DSIC01LS-P_C600988, SW4 DSIC01LS-P_C600988, SW5 DSIC01LS-P_C600988, U1 ADS131E08IPAGR, U2 DB125-2.54-2P-GN, U4 TPS61299DRLR, U5 TPS7A2050PDBVR, U6 PM2.54-YP1D-14A, U7 PM2.54-YP1D-14A, U8 PM2.54-YP1D-14A, U9 PM2.54-YP1D-14A

Commit message: recover tempoary data file
Parts:
- added C33: 10uF, Capacitor_SMD:C_0603_1608Metric, F.Cu at (47.6, 52.6)
- added U10: DB125-2.54-2P-GN, easyeda2kicad:CONN-TH_DB125-2.54-2P-GN, F.Cu at (40.0, 94.0)
- moved C24 3.30 mm to (40.6, 34.5)
- moved C25 3.30 mm to (49.2, 34.0)
- moved C26 3.30 mm to (52.1, 34.5)
- moved C27 3.30 mm to (53.9, 36.0)
- moved C28 3.30 mm to (60.9, 36.0)
- moved L1 3.30 mm to (45.0, 35.3)
- moved NT1 3.30 mm to (52.9, 40.0)
- moved R17 3.30 mm to (51.9, 37.5)
- moved SW2 3.30 mm to (54.9, 46.8)
- moved SW3 3.30 mm to (43.1, 49.3)
- moved U4 3.30 mm to (49.4, 35.9)
- moved U5 3.30 mm to (57.3, 36.1)
- moved U7 2.54 mm to (62.2, 94.0)
- moved U8 2.54 mm to (62.2, 78.7)
- moved U6 2.54 mm to (62.2, 76.2)
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Connections:
- U1 pad 24: /adcAVSS -> /adcREF+
- U1 pad 25: /adcREF+ -> /adcAVSS
- U1 pad 52: GNDD -> +3.3V
Routing:
- net VCC: track 43.3 -> 62.8 mm
- net +3.3V: track 71.3 -> 78.4 mm, vias 1 -> 4
- net /adcAVSS: track 30.6 -> 33.5 mm
- net /CS: track 65.0 -> 67.9 mm
- net GNDD: track 32.7 -> 29.9 mm, vias 33 -> 41
- net /SPI_MOSI: track 73.7 -> 76.3 mm
- net /SPI_CLK: track 62.0 -> 64.5 mm
- net /FLC100_connector2/OUT-: track 30.8 -> 28.7 mm
- net /FLC100_connector3/OUT-: track 45.5 -> 43.6 mm
- net /adcAVDD: track 239.6 -> 238.0 mm
- net Net-(U1-IN4P): vias 1 -> 0
Other:
- board size 99 x 69 mm -> 98.9 x 66.8 mm
- board text added: "2.5V ref"
- board text added: "5V bypass"
- board text added: "5V smoothing on"
- board text added: "Battery/power input port? Solar charger?"
- board text added: "CS"
- board text added: "GND"
- board text added: "MISO"
- board text added: "MOSI"
- board text added: "SCLK"
- board text added: "SMACT FLC100 v0.1"
- board text added: "nDRDY"
- board text removed: "SMACT FLC100 v0"
