File: FLC100_pcb/FLC100_pcb.kicad_sch (KiCad schematic)
At the start: 42 parts, among them SW2 DSIC01LS-P_C600988, SW3 DSIC01LS-P_C600988, SW4 DSIC01LS-P_C600988, SW5 DSIC01LS-P_C600988, U1 ADS131E08IPAGR, U2 DB125-2.54-2P-GN, U6 PM2.54-YP1D-14A, U7 PM2.54-YP1D-14A, U8 PM2.54-YP1D-14A, U9 PM2.54-YP1D-14A

Commit message: recover tempoary data file
Parts:
- added C33: 10uF, Capacitor_SMD:C_0603_1608Metric, symbol Device:C
- added U10: DB125-2.54-2P-GN, easyeda2kicad:CONN-TH_DB125-2.54-2P-GN, symbol easyeda:DB125-2.54-2P-GN
Connections:
- net +3.3V: now also U1.52 (CLKSEL)
- net GNDD: now also C33.2, U10.1; no longer U1.52 (CLKSEL)
- net VCC: now also C33.1, U10.2
- net adcAVSS: now also U1.25 (VREFN); no longer U1.24 (VREFP)
- net adcREF+: now also U1.24 (VREFP); no longer U1.25 (VREFN)
